File: XmasTree.brd (EAGLE design)
At the start: 40 x 40 mm, 26 parts, among them Q1 MUN5235DW1T1G, Q2 MUN5235DW1T1G, U1 MCP1640C, U2 ATtiny84A-SSU

Commit message: Add select button.
Parts:
- added S2: SELECT, _jc:B3F-10XXOCT
- moved LOGO1 9.12 mm to (31.4, 7.50)
- moved LOGO2 9.12 mm to (35.9, 7.50)
Connections:
- new net N$12: S2.1, S2.2, U2.12
- net GND: now also S2.3, S2.4
Routing:
- net N$12: track 0.00 -> 40.0 mm, vias 0 -> 1
Changed lines of the file:
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@@
 <text x="12" y="1.5" size="2.1844" layer="21" ratio="16" align="bottom-center">OFF</text>
 <text x="27.5" y="1.5" size="2.1844" layer="21" ratio="16" align="bottom-center">ON</text>
-<text x="35" y="15" size="1.016" layer="21" ratio="16" align="bottom-center">open source</text>
-<text x="31" y="7.5" size="1.016" layer="21" ratio="16" align="bottom-center">Xmas Tree LEDs v1.0
+<text x="33.5" y="6" size="1.016" layer="21" ratio="16" align="bottom-center">open source</text>
+<text x="20" y="6" size="1.016" layer="21" ratio="16" align="bottom-center">Xmas Tree LEDs v1.0
 CC BY-SA 4.0 jc 1123
 bit.ly/xtleds</text>
-<text x="35" y="15" size="1.016" layer="22" ratio="16" rot="MR0" align="bottom-center">open source</text>
-<text x="31" y="7.5" size="1.016" layer="22" ratio="16" rot="MR0" align="bottom-center">Xmas Tree LEDs v1.0
+<text x="33.5" y="6" size="1.016" layer="22" ratio="16" rot="MR0" align="bottom-center">open source</text>
+<text x="20" y="6" size="1.016" layer="22" ratio="16" rot="MR0" align="bottom-center">Xmas Tree LEDs v1.0
 CC BY-SA 4.0 jc 1123
 bit.ly/xtleds</text>
@@
 <attribute name="VALUE" x="5.63" y="3.07" size="1.016" layer="27" ratio="10"/>
 </element>
-<element name="LOGO1" library="ohw-logo" package="OSHW_8X150_NOTEXT" value="OSHW_LOGO_8MILX0150-NT" x="32.94" y="16.5" smashed="yes"/>
-<element name="LOGO2" library="ohw-logo" package="OSHW_8X150_NOTEXT" value="OSHW_LOGO_8MILX0150-NT" x="37.36" y="16.5" smashed="yes" rot="MR0"/>
+<element name="LOGO1" library="ohw-logo" package="OSHW_8X150_NOTEXT" value="OSHW_LOGO_8MILX0150-NT" x="31.44" y="7.5" smashed="yes"/>
+<element name="LOGO2" library="ohw-logo" package="OSHW_8X150_NOTEXT" value="OSHW_LOGO_8MILX0150-NT" x="35.86" y="7.5" smashed="yes" rot="MR0"/>
 <element name="Q1" library="_jc" package="SOT363_PHILIPS" value="MUN5235DW1T1G" x="20" y="20" smashed="yes" rot="R270">
 <attribute name="NAME" x="19.4" y="17.85" size="0.8128" layer="25" ratio="16"/>
@@
 <attribute name="NAME" x="17.9" y="38.5" size="0.8128" layer="25" ratio="16"/>
 <attribute name="VALUE" x="17" y="34.5" size="0.8128" layer="27" ratio="16"/>
+</element>
+<element name="S2" library="_jc" package="B3F-10XXOCT" value="SELECT" x="35" y="17.5" smashed="yes" rot="R90">
+<attribute name="NAME" x="34.452" y="17.183" size="0.8128" layer="25" ratio="16"/>
+<attribute name="VALUE" x="40.08" y="14.452" size="1.27" layer="27" ratio="16" rot="R90"/>
 </element>
 </elements>
@@
 <contactref element="JP2" pad="2"/>
 <polygon width="0.254" layer="1" isolate="0.254">
-<vertex x="-1" y="-1"/>
-<vertex x="41" y="-1"/>
-<vertex x="41" y="41"/>
-<vertex x="-1" y="41"/>
+<vertex x="-1.5" y="-1.5"/>
+<vertex x="41.5" y="-1.5"/>
+<vertex x="41.5" y="41.5"/>
+<vertex x="-1.5" y="41.5"/>
 </polygon>
 <contactref element="R8" pad="2"/>
+<contactref element="S2" pad="4"/>
+<contactref element="S2" pad="3"/>
 </signal>
 <signal name="N$7">
@@
 <contactref element="JP1" pad="2"/>
 <polygon width="0.254" layer="16" isolate="0.254">
-<vertex x="-0.5" y="-0.5"/>
-<vertex x="40.5" y="-0.5"/>
-<vertex x="40.5" y="40.5"/>
-<vertex x="-0.5" y="40.5"/>
+<vertex x="-1" y="-1"/>
+<vertex x="41" y="-1"/>
+<vertex x="41" y="41"/>
+<vertex x="-1" y="41"/>
 </polygon>
 <via x="9" y="19.5" extent="1-16" drill="0.8" shape="octagon"/>
@@
 <wire x1="11.45" y1="35.97" x2="11.45" y2="34.45" width="0.254" layer="1"/>
 <wire x1="11.45" y1="34.45" x2="11.2" y2="34.2" width="0.254" layer="1"/>
-<wire x1="9.7" y1="34.2" x2="9" y2="33.5" width="0.254" layer="1"/>
-<via x="9" y="33.5" extent="1-16" drill="0.35" shape="octagon"/>
-<wire x1="9" y1="33.5" x2="9" y2="24.4" width="0.254" layer="16"/>
-<wire x1="11.2" y1="34.2" x2="9.7" y2="34.2" width="0.254" layer="1"/>
+<wire x1="9" y1="24.4" x2="9" y2="33" width="0.254" layer="16"/>
+<wire x1="11.2" y1="34.2" x2="10.5" y2="34.2" width="0.254" layer="1"/>
 <via x="9" y="24.4" extent="1-16" drill="0.35" shape="octagon"/>
 <wire x1="11" y1="22.4" x2="9" y2="24.4" width="0.254" layer="1"/>
@@
 <wire x1="10.5" y1="14.4" x2="11" y2="14.9" width="0.254" layer="1"/>
 <wire x1="11" y1="14.9" x2="11" y2="22.4" width="0.254" layer="1"/>
+<via x="9" y="33" extent="1-16" drill="0.35" shape="octagon"/>
+<wire x1="9" y1="33" x2="10.2" y2="34.2" width="0.254" layer="1"/>
+<wire x1="10.2" y1="34.2" x2="10.5" y2="34.2" width="0.254" layer="1"/>
 </signal>
 <signal name="N$6">
@@
 <wire x1="10.5" y1="38" x2="15.5" y2="38" width="0.254" layer="1"/>
 </signal>
+<signal name="N$12">
+<contactref element="U2" pad="12"/>
+<contactref element="S2" pad="1"/>
+<contactref element="S2" pad="2"/>
+<wire x1="8.91" y1="35.97" x2="8.91" y2="34.41" width="0.254" layer="1"/>
+<wire x1="8.91" y1="34.41" x2="8.5" y2="34" width="0.254" layer="1"/>
+<wire x1="8.5" y1="34" x2="8" y2="34" width="0.254" layer="1"/>
+<via x="8" y="34" extent="1-16" drill="0.35" shape="octagon"/>
+<wire x1="8" y1="34" x2="9.5" y2="34" width="0.254" layer="16"/>
+<wire x1="32.7394" y1="20.7512" x2="32.7394" y2="14.2488" width="0.254" layer="16"/>
+<wire x1="15" y1="28.5" x2="15" y2="27.5" width="0.254" layer="16"/>
+<wire x1="15" y1="27.5" x2="19.5" y2="23" width="0.254" layer="16"/>
+<wire x1="30.4906" y1="23" x2="32.7394" y2="20.7512" width="0.254" layer="16"/>
+<wire x1="9.5" y1="34" x2="15" y2="28.5" width="0.254" layer="16"/>
+<wire x1="19.5" y1="23" x2="30.4906" y2="23" width="0.254" layer="16"/>
+</signal>
 </signals>

Commit message: Update LED dropping resistor values.
Parts:
- R1, R2, R3, R4: value 62 -> 15
Changed lines of the file:
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@@
 <attribute name="VALUE" x="17.37" y="32.18" size="0.8128" layer="27" ratio="16" rot="R270"/>
 </element>
-<element name="R1" library="_jc" package="M0805" value="62" x="15.61" y="14.04" smashed="yes" rot="R90">
+<element name="R1" library="_jc" package="M0805" value="15" x="15.61" y="14.04" smashed="yes" rot="R90">
 <attribute name="NAME" x="14.11" y="12.54" size="0.8128" layer="25" ratio="16" rot="R90"/>
 <attribute name="VALUE" x="18.11" y="12.54" size="0.8128" layer="27" ratio="16" rot="R90"/>
 </element>
-<element name="R2" library="_jc" package="M0805" value="62" x="26.14" y="15.61" smashed="yes" rot="R180">
+<element name="R2" library="_jc" package="M0805" value="15" x="26.14" y="15.61" smashed="yes" rot="R180">
 <attribute name="NAME" x="27.64" y="14.11" size="0.8128" layer="25" ratio="16" rot="R180"/>
 <attribute name="VALUE" x="27.64" y="18.11" size="0.8128" layer="27" ratio="16" rot="R180"/>
 </element>
-<element name="R3" library="_jc" package="M0805" value="62" x="24.41" y="25.98" smashed="yes" rot="R90">
+<element name="R3" library="_jc" package="M0805" value="15" x="24.41" y="25.98" smashed="yes" rot="R90">
 <attribute name="NAME" x="24.98" y="28.29" size="0.8128" layer="25" ratio="16"/>
 <attribute name="VALUE" x="26.91" y="24.48" size="0.8128" layer="27" ratio="16" rot="R90"/>
 </element>
-<element name="R4" library="_jc" package="M0805" value="62" x="14" y="24.39" smashed="yes">
+<element name="R4" library="_jc" package="M0805" value="15" x="14" y="24.39" smashed="yes">
 <attribute name="NAME" x="12.5" y="25.89" size="0.8128" layer="25" ratio="16"/>
 <attribute name="VALUE" x="12.5" y="21.89" size="0.8128" layer="27" ratio="16"/>

Commit message: Board tweaks.
Routing:
- net MOSI/SDA: track 21.2 -> 23.2 mm
- net VIN: track 22.0 -> 22.8 mm
Other:
- board text added: "Xmas Tree LEDs v1.1 CC BY-SA 4.0 jc 1223 bit.ly/xtleds"
- board text removed: "Xmas Tree LEDs v1.0 CC BY-SA 4.0 jc 1123 bit.ly/xtleds"
Changed lines of the file:
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@@
 <wire x1="28" y1="40" x2="12" y2="40" width="0" layer="20"/>
 <wire x1="12" y1="40" x2="0" y2="28" width="0" layer="20" curve="90"/>
-<hole x="28" y="25" drill="2.5"/>
-<circle x="28" y="25" radius="1.5" width="0" layer="41"/>
-<circle x="28" y="25" radius="1.5" width="0" layer="42"/>
+<hole x="28" y="25" drill="3"/>
+<circle x="28" y="25" radius="1.75" width="0" layer="41"/>
+<circle x="28" y="25" radius="1.75" width="0" layer="42"/>
 <text x="38.5" y="25" size="1.016" layer="21" ratio="16" rot="R90" align="bottom-center">+3VDC-</text>
 <text x="31" y="30" size="1.016" layer="21" ratio="16" align="bottom-center">ICSP</text>
@@
 <text x="27.5" y="1.5" size="2.1844" layer="21" ratio="16" align="bottom-center">ON</text>
 <text x="33.5" y="6" size="1.016" layer="21" ratio="16" align="bottom-center">open source</text>
-<text x="20" y="6" size="1.016" layer="21" ratio="16" align="bottom-center">Xmas Tree LEDs v1.0
-CC BY-SA 4.0 jc 1123
+<text x="20" y="6" size="1.016" layer="21" ratio="16" align="bottom-center">Xmas Tree LEDs v1.1
+CC BY-SA 4.0 jc 1223
 bit.ly/xtleds</text>
 <text x="33.5" y="6" size="1.016" layer="22" ratio="16" rot="MR0" align="bottom-center">open source</text>
-<text x="20" y="6" size="1.016" layer="22" ratio="16" rot="MR0" align="bottom-center">Xmas Tree LEDs v1.0
-CC BY-SA 4.0 jc 1123
+<text x="20" y="6" size="1.016" layer="22" ratio="16" rot="MR0" align="bottom-center">Xmas Tree LEDs v1.1
+CC BY-SA 4.0 jc 1223
 bit.ly/xtleds</text>
 </plain>
@@
 <wire x1="6.6" y1="10.4" x2="6.81" y2="10.19" width="0.3048" layer="1"/>
 <wire x1="6.81" y1="10.19" x2="7.11" y2="10.19" width="0.3048" layer="1"/>
-<wire x1="6.63" y1="7.07" x2="6.63" y2="4.97" width="0.508" layer="1"/>
-<wire x1="6.63" y1="4.97" x2="7.2" y2="4.4" width="0.508" layer="1"/>
+<wire x1="6.63" y1="4.97" x2="6.63" y2="7.07" width="0.508" layer="1"/>
 <contactref element="S1" pad="P$2"/>
-<wire x1="20" y1="4.4" x2="7.2" y2="4.4" width="0.508" layer="1"/>
 <wire x1="7.11" y1="10.19" x2="7" y2="10.08" width="0.3048" layer="1"/>
 <wire x1="7" y1="7.44" x2="6.63" y2="7.07" width="0.3048" layer="1"/>
 <wire x1="7" y1="10.08" x2="7" y2="7.44" width="0.3048" layer="1"/>
+<wire x1="20" y1="4.4" x2="19.1" y2="3.5" width="0.508" layer="1"/>
+<wire x1="19.1" y1="3.5" x2="8.1" y2="3.5" width="0.508" layer="1"/>
+<wire x1="8.1" y1="3.5" x2="6.63" y2="4.97" width="0.508" layer="1"/>
 </signal>
 <signal name="GND">
@@
 <wire x1="28.636" y1="31" x2="30.75" y2="33.114" width="0.254" layer="16"/>
 <wire x1="24.5" y1="32" x2="23.7" y2="32.8" width="0.254" layer="1"/>
-<wire x1="18.97" y1="31.08" x2="18" y2="31.08" width="0.254" layer="1"/>
-<wire x1="18" y1="31.08" x2="13.99" y2="31.08" width="0.254" layer="1"/>
-<wire x1="13.99" y1="31.08" x2="13.99" y2="30.77" width="0.254" layer="1"/>
-<wire x1="23.7" y1="32.8" x2="18.3" y2="32.8" width="0.254" layer="1"/>
-<wire x1="18.3" y1="32.8" x2="18" y2="32.5" width="0.254" layer="1"/>
-<wire x1="18" y1="32.5" x2="18" y2="31.08" width="0.254" layer="1"/>
+<wire x1="13.99" y1="32.49" x2="13.99" y2="30.77" width="0.254" layer="1"/>
+<wire x1="23.7" y1="32.8" x2="17.5" y2="32.8" width="0.254" layer="1"/>
+<wire x1="17.5" y1="32.8" x2="14.3" y2="32.8" width="0.254" layer="1"/>
+<wire x1="14.3" y1="32.8" x2="13.99" y2="32.49" width="0.254" layer="1"/>
+<wire x1="18.97" y1="31.08" x2="18.89" y2="31" width="0.254" layer="1"/>
+<wire x1="18.89" y1="31" x2="18" y2="31" width="0.254" layer="1"/>
+<wire x1="18" y1="31" x2="17.5" y2="31.5" width="0.254" layer="1"/>
+<wire x1="17.5" y1="31.5" x2="17.5" y2="32.8" width="0.254" layer="1"/>
 </signal>
 <signal name="PB2">
@@
 <wire x1="15" y1="28.5" x2="15" y2="27.5" width="0.254" layer="16"/>
 <wire x1="15" y1="27.5" x2="19.5" y2="23" width="0.254" layer="16"/>
-<wire x1="30.4906" y1="23" x2="32.7394" y2="20.7512" width="0.254" layer="16"/>
 <wire x1="9.5" y1="34" x2="15" y2="28.5" width="0.254" layer="16"/>
-<wire x1="19.5" y1="23" x2="30.4906" y2="23" width="0.254" layer="16"/>
+<wire x1="26.5" y1="23" x2="19.5" y2="23" width="0.254" layer="16"/>
+<wire x1="32.7394" y1="20.7512" x2="28.7488" y2="20.7512" width="0.254" layer="16"/>
+<wire x1="28.7488" y1="20.7512" x2="26.5" y2="23" width="0.254" layer="16"/>
 </signal>
 </signals>

Commit message: Cosmetic tweaks to schematic.
Parts:
- Q1, Q2: value MUN5235DW1T1G -> MUN5235DW1
Changed lines of the file:
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@@
 <element name="LOGO1" library="ohw-logo" package="OSHW_8X150_NOTEXT" value="OSHW_LOGO_8MILX0150-NT" x="31.44" y="7.5" smashed="yes"/>
 <element name="LOGO2" library="ohw-logo" package="OSHW_8X150_NOTEXT" value="OSHW_LOGO_8MILX0150-NT" x="35.86" y="7.5" smashed="yes" rot="MR0"/>
-<element name="Q1" library="_jc" package="SOT363_PHILIPS" value="MUN5235DW1T1G" x="20" y="20" smashed="yes" rot="R270">
+<element name="Q1" library="_jc" package="SOT363_PHILIPS" value="MUN5235DW1" x="20" y="20" smashed="yes" rot="R270">
 <attribute name="NAME" x="19.4" y="17.85" size="0.8128" layer="25" ratio="16"/>
 <attribute name="VALUE" x="17.3" y="21.1" size="0.8128" layer="27" ratio="16" rot="R270"/>
 </element>
-<element name="Q2" library="_jc" package="SOT363_PHILIPS" value="MUN5235DW1T1G" x="20.07" y="31.08" smashed="yes" rot="R270">
+<element name="Q2" library="_jc" package="SOT363_PHILIPS" value="MUN5235DW1" x="20.07" y="31.08" smashed="yes" rot="R270">
 <attribute name="NAME" x="19.52" y="32.42" size="0.8128" layer="25" ratio="16"/>
 <attribute name="VALUE" x="17.37" y="32.18" size="0.8128" layer="27" ratio="16" rot="R270"/>
